File: hardware/PCB/KiCad/Macro-Keyboard-v4/Macro-Keyboard-v4.kicad_sch (KiCad schematic)
At the start: 40 parts, among them IC1 AS5600-ASOT, J2 OLED_128x64, J3 5VUSB-PIN+, J4 5VUSB-PIN-, J5 JST_03, J6 Conn_ARM_JTAG_SWD_10, SW1 POWER-SWITCH, SW4 RESET, U2 USBLC6-2SC6, U4 BQ24040DSQR, U6 MDBT50Q-1MV2, X1 Q13FC1350000400

Commit message: Adding BOMs and PCB(A) production files
Parts:
- J2: now in the parts list
- J3, J4, J6: now left out of the parts list
